File: hardware/bbb_d300_cape.sch (EAGLE design)
At the start: 38 parts, among them IC1 7414D, IC2 7414D, T1 2N3904, T2 2N3904, T3 2N3904, T4 2N3904, T5 2N3904

Commit message: connect tool length to P8.08
Signed-off-by: Vladimir Pantelic <vladimir@pantelic.net>
Connections:
- net ERR3 renamed ERR3V3
- net HOME3 renamed HOME3V3
- removed net LENGTH3: PCB2.P8.11, R16.1, T3.C
- new net LENGTH3V3: PCB2.P8.8, R16.1, T3.C
Changed lines of the file:
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@@
 </segment>
 </net>
-<net name="ERR3" class="0">
+<net name="ERR3V3" class="0">
 <segment>
 <pinref part="R4" gate="G$1" pin="1"/>
@@
 <wire x1="269.24" y1="147.32" x2="269.24" y2="142.24" width="0.1524" layer="91"/>
 <wire x1="269.24" y1="142.24" x2="254" y2="142.24" width="0.1524" layer="91"/>
-<label x="254" y="142.24" size="1.778" layer="95"/>
+<label x="251.46" y="142.24" size="1.778" layer="95"/>
 <junction x="269.24" y="142.24"/>
 </segment>
@@
 </segment>
 </net>
-<net name="HOME3" class="0">
+<net name="HOME3V3" class="0">
 <segment>
 <pinref part="R3" gate="G$1" pin="1"/>
@@
 </segment>
 </net>
-<net name="LENGTH3" class="0">
+<net name="LENGTH3V3" class="0">
 <segment>
 <pinref part="R16" gate="G$1" pin="1"/>
@@
 </segment>
 <segment>
-<pinref part="PCB2" gate="G$1" pin="P8.11"/>
-<wire x1="129.54" y1="114.3" x2="134.62" y2="114.3" width="0.1524" layer="91"/>
-<label x="132.08" y="114.3" size="1.778" layer="95"/>
+<pinref part="PCB2" gate="G$1" pin="P8.8"/>
+<wire x1="129.54" y1="121.92" x2="134.62" y2="121.92" width="0.1524" layer="91"/>
+<label x="132.08" y="121.92" size="1.778" layer="95"/>
 </segment>
 </net>
@@
 <wire x1="269.24" y1="63.5" x2="269.24" y2="58.42" width="0.1524" layer="91"/>
 <wire x1="269.24" y1="58.42" x2="254" y2="58.42" width="0.1524" layer="91"/>
-<label x="251.46" y="58.42" size="1.778" layer="95"/>
+<label x="254" y="58.42" size="1.778" layer="95"/>
 <pinref part="TP11" gate="G$1" pin="TP"/>
 <junction x="269.24" y="58.42"/>
